File: testBoard.kicad_pcb (KiCad board)
At the start: 2 copper layers, 96 x 96 mm, 75 parts, among them J1 Conn_02x05_Odd_Even, J2 Conn_01x06, J3 Conn_01x02, Q1 SCT2450KEC, SW1 PTS645SM43SMTR92_LFS, U1 PIC18F47K40, U10 INA233, U11 INA233, U12 TPS2557, U13 EMCO-Q50-5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

Commit message: Hopefully fixed pins
Parts:
- D1: value PWR -> LED_ALT
- D2: value RDY -> LED_RDY
- D3, D5: value DIA -> LED_DIA
- D4: value ERR -> LED_ERR
- J3: value Conn_01x02 -> Thruster_Connection
Connections:
- net Net-(CD1-Pad1) renamed /CAP_BANK_POSITIVE
- net Net-(J3-Pad1) renamed /Thruster_Control
- net RA5 renamed THRUST_CONTROL
- U1 pad 19: U4_EN -> U12_FAULT
- U1 pad 2: U12_EN -> U4_EN
- U1 pad 20: Net-(D2-Pad2) -> U14_FAULT
- U1 pad 21: Net-(D4-Pad2) -> U12_EN
- U1 pad 22: Net-(D5-Pad2) -> U14_EN
- U1 pad 3: U14_EN -> Net-(D2-Pad2)
- U1 pad 4: U12_FAULT -> Net-(D4-Pad2)
- U1 pad 5: U14_FAULT -> Net-(D5-Pad2)
