File: testBoard.kicad_pcb (KiCad board)
At the start: 2 copper layers, 88 x 96 mm, 75 parts, among them J1 Conn_02x05_Odd_Even, J2 Conn_01x06, J3 Thruster_Connection, Q1 SCT2450KEC, SW1 PTS645SM43SMTR92_LFS, U1 PIC18F47K40, U10 INA233, U11 INA233, U12 TPS2557, U13 EMCO-Q50-5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

Commit message: Final board design
Parts:
- RSCL1, RSDA1: moved to B.Cu
- U13, U15, U6: footprint PPTBoard:EMCO_Q_2.5-5kV -> PPTBoard:EMCO_Q_2.5-5kV-Shielded
- moved COUT1 37.5 mm to (143.3, 82.5)
- moved RSCL2 31.0 mm to (141.1, 71.8), turned to 180 degrees
- moved DISCP1 15.9 mm to (107.7, 57.7), turned to 180 degrees
- moved RIS4 15.8 mm to (143.8, 116.8), turned to 0 degrees
- moved U2 9.03 mm to (112.0, 52.1), turned to 180 degrees
- moved RSDA2 8.51 mm to (119.4, 73.4)
- moved SW1 8.14 mm to (120.1, 52.8), turned to 180 degrees
- moved RF2 7.15 mm to (127.3, 61.5), turned to 90 degrees
- moved RF1 5.08 mm to (151.9, 104.6), turned to 0 degrees
- moved RMCLR1 4.57 mm to (114.0, 57.9), turned to 180 degrees
- moved RILIM1 4.49 mm to (150.4, 111.3), turned to 180 degrees
- moved RAL4 3.05 mm to (140.7, 107.7)
- moved U10 3.05 mm to (140.7, 111.0)
- moved COUT2 2.17 mm to (139.2, 101.3)
- moved RAL1 2.05 mm to (118.1, 102.1)
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Connections:
- net /Thruster_Control renamed /Thrust_Connector
- U1 pad 10: SDA2 -> SDA1
- U1 pad 15: (no net) -> U9_ALERT
- U1 pad 19: U9_ALERT -> U3_EN
- U1 pad 21: U12_FAULT -> U12_EN
- U1 pad 22: U12_EN -> U12_FAULT
- U1 pad 23: U3_EN -> U5_DIN
- U1 pad 24: U4_EN -> SCLK
- U1 pad 25: U5_DIN -> U5_CS
- U1 pad 26: SCLK -> U4_EN
- U1 pad 30: U5_CS -> (no net)
- U1 pad 37: SCL1 -> SCL2
- U1 pad 42: SDA1 -> SDA2
- U1 pad 43: THRUST_CONTROL -> U16_CS
- U1 pad 44: U16_CS -> THRUST_CONTROL
- U1 pad 9: SCL2 -> SCL1
Routing:
- net GND: track 224.4 -> 43.5 mm, vias 17 -> 2
- net VCC: track 328.7 -> 299.3 mm, vias 21 -> 8
- net SDA1: track 75.6 -> 56.5 mm, vias 4 -> 1
- net SCL2: track 111.6 -> 94.3 mm, vias 9 -> 5
- net SCL1: track 69.0 -> 52.8 mm, vias 3 -> 1
- net /U12_VOUT: track 42.1 -> 26.7 mm, vias 2 -> 0
- net /U6_VIN: track 39.5 -> 27.3 mm, vias 2 -> 1
- net U4_VOUT: track 50.3 -> 61.7 mm, vias 2 -> 0
- net SDA2: track 101.3 -> 92.4 mm, vias 12 -> 5
- net U12_FAULT: track 43.1 -> 35.6 mm, vias 4 -> 0
- net U10_ALERT: track 32.5 -> 38.3 mm, vias 2 -> 0
- net PM_VIN: track 60.3 -> 66.0 mm
- net U3_EN: track 49.0 -> 43.5 mm
- net U5_CS: track 30.2 -> 24.9 mm
- net MCLR: track 51.4 -> 46.7 mm, vias 2 -> 1
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Other:
- net class 10mil: clearance 0 -> 0.127
- net class 12mil: clearance 0 -> 0.254
- net class 20mil: clearance 0 -> 0.254
- net class 40mil: clearance 0 -> 0.254
- net class 60mil: clearance 0 -> 0.254
- net class Default: clearance 0 -> 0.0635
- rule trace_clearance: 0 -> 0.0635
