File: testBoard.sch (KiCad schematic (older format))
At the start: 75 parts, among them J1 Conn_02x05_Odd_Even, J2 Conn_01x06, J3 Thruster_Connection, Q1 SCT2450KEC, SW1 PTS645SM43SMTR92_LFS, U1 PIC18F47K40, U10 INA233, U11 INA233, U12 TPS2557, U13 EMCO-Q50-5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

Commit message: Hopefully fixed pins
Connections:
- net U12_EN: now also U1.21 (RA2); no longer U1.2 (RD4)
- net U12_FAULT: now also U1.19 (RA0); no longer U1.4 (RD6)
- net U14_EN: now also U1.22 (RA3); no longer U1.3 (RD5)
- net U14_FAULT: now also U1.20 (RA1); no longer U1.5 (RD7)
- net U4_EN: now also U1.2 (RD4); no longer U1.19 (RA0)
- net at D2.2 (A): now also U1.3 (RD5); no longer U1.20 (RA1)
- net at D4.2 (A): now also U1.4 (RD6); no longer U1.21 (RA2)
- net at D5.2 (A): now also U1.5 (RD7); no longer U1.22 (RA3)
- net RA5 renamed THRUST_CONTROL
Other:
- moved on the sheet: CSPK2, D2, D4, D5, Q1, RAL5, RF2, RILIM2, RIS5, RLED2, RLED4, RLED5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

Commit message: Board design 1
Parts:
- CSPK1, CSPK2: footprint Capacitor_SMD:C_Elec_6.3x7.7 -> Capacitor_SMD:C_2220_5650Metric
- D1: value LED_ALT -> PWR
- D2: value LED_RDY -> RDY
- D3: value LED_DIA -> DIA2
- D4: value LED_ERR -> ERR
- D5: value LED_DIA -> DIA
Connections:
- net SCL1: now also J1.4 (Pin_4)
- net SCLK: now also U1.26 (RE1); no longer U1.40 (RD2)
- net SDA1: now also J1.6 (Pin_6)
- net THRUST_CONTROL: now also U1.43 (RC5); no longer U1.24 (RA5)
- net U10_ALERT: now also U1.20 (RA1); no longer U1.36 (RC2)
- net U11_ALERT: now also U1.32 (RC0); no longer U1.43 (RC5)
- net U12_EN: now also U1.22 (RA3); no longer U1.21 (RA2)
- net U12_FAULT: now also U1.21 (RA2); no longer U1.19 (RA0)
- net U14_EN: now also U1.35 (RC1); no longer U1.22 (RA3)
- net U14_FAULT: now also U1.36 (RC2); no longer U1.20 (RA1)
- net U4_EN: now also U1.24 (RA5); no longer U1.2 (RD4)
- net U5_CS: now also U1.30 (RA7); no longer U1.41 (RD3)
- net U5_DIN: now also U1.25 (RE0); no longer U1.39 (RD1)
- net U7_ALERT: now also U1.14 (RB4); no longer U1.11 (RB3)
- net U8_ALERT: now also U1.11 (RB3); no longer U1.14 (RB4)
- net U9_ALERT: now also U1.19 (RA0); no longer U1.15 (RB5)
- net DIA_LED: now reaches U1.1 (RC7)
- net DIA_LED: now also D5.2 (A)
- net U3_EN: now reaches U1.23 (RA4)
- net U3_EN: now also U3.3 (EN)
- net ERR_LED: now reaches U1.3 (RD5)
- net ERR_LED: now also D4.2 (A); no longer D2.2 (A)
- net DIA2_LED: now reaches D3.2 (A)
- net DIA2_LED: now also U1.2 (RD4); no longer U1.32 (RC0)
- net RDY_LED: now reaches U1.4 (RD6)
- net RDY_LED: now also D2.2 (A); no longer D4.2 (A)
- net at U1.5 (RD7): no longer D5.2 (A)
- net U12_ILIM: now reaches RILIM1.1, U12.5 (ILM)
- net U12_VOUT: now reaches RIS4.2, U10.10 (IN+), U12.6 (OUT), U12.7 (OUT)
- net U14_ILIM: now reaches RILIM2.1, U14.5 (ILM)
- net U14_OUT: now reaches RIS5.1, U11.10 (IN+), U14.6 (OUT), U14.7 (OUT)
- net U7_DIAG_NET: now reaches J1.1 (Pin_1), J1.2 (Pin_2), RIS1.1, U7.10 (IN+)
- net U6_VIN: now reaches RIS3.2, U6.2 ((+)IN), U9.8 (VBUS), U9.9 (IN-)
- net DBNC_DDE_PRTCTD: now reaches DISCP1.1 (K), RMCLR1.2, U2.3 (OUT)
- net R_DIA2: now reaches D3.1 (K), RLED3.2
- net R_RDY: now reaches D2.1 (K), RLED2.2
- net R_ERR: now reaches D4.1 (K), RLED4.2
- net R_DIA: now reaches D5.1 (K), RLED5.2
- net TC-: now reaches TC1.2 (-), U16.2 (T-)
- net TC+: now reaches TC1.1 (+), U16.3 (T+)
- net U15_VIN: now reaches RIS5.2, U11.8 (VBUS), U11.9 (IN-), U15.2 ((+)IN)
- net SPK2: now reaches CSPK2.1, U15.3 (HV_OUTPUT)
- net U4_FB: now reaches RFBB2.1, U4.5 (FB), U5.10 (L)
- net U13_VIN: now reaches RIS4.1, U10.8 (VBUS), U10.9 (IN-), U13.2 ((+)IN)
- net SPK1: now reaches CSPK1.1, U13.3 (HV_OUTPUT)
- net U3-FB: now reaches RFBB1.1, RFBT1.2, U3.5 (FB)
- no-connect marks 21 -> 9
Other:
- note added: "Check w/\n Dr. White\n if needed"
- moved on the sheet: D1, D2, D3, D4, D5, RLED1, RLED2, RLED3, RLED4, RLED5

Commit message: Final board design
Parts:
- U13, U15, U6: footprint PPTBoard:EMCO_Q_2.5-5kV -> PPTBoard:EMCO_Q_2.5-5kV-Shielded
Connections:
- net GND: now also U13.8 (SHIELD), U15.8 (SHIELD), U6.8 (SHIELD)
- net SCL1: now also U1.9 (RB1); no longer U1.37 (RC3)
- net SCL2: now also U1.37 (RC3); no longer U1.9 (RB1)
- net SCLK: now also U1.24 (RA5); no longer U1.26 (RE1)
- net SDA1: now also U1.10 (RB2); no longer U1.42 (RC4)
- net SDA2: now also U1.42 (RC4); no longer U1.10 (RB2)
- net THRUST_CONTROL: now also U1.44 (RC6); no longer U1.43 (RC5)
- net U12_EN: now also U1.21 (RA2); no longer U1.22 (RA3)
- net U12_FAULT: now also U1.22 (RA3); no longer U1.21 (RA2)
- net U16_CS: now also U1.43 (RC5); no longer U1.44 (RC6)
- net U3_EN: now also U1.19 (RA0); no longer U1.23 (RA4)
- net U4_EN: now also U1.26 (RE1); no longer U1.24 (RA5)
- net U5_CS: now also U1.25 (RE0); no longer U1.30 (RA7)
- net U5_DIN: now also U1.23 (RA4); no longer U1.25 (RE0)
- net U9_ALERT: now also U1.15 (RB5); no longer U1.19 (RA0)
- net Thruster_Control renamed Thrust_Connector
Changed lines of the file:
@@
 F 0 "U13" H 4950 9217 50  0000 C CNN
 F 1 "EMCO-Q50-5" H 4950 9126 50  0000 C CNN
-F 2 "PPTBoard:EMCO_Q_2.5-5kV" H 4350 8950 50  0001 C CNN
+F 2 "PPTBoard:EMCO_Q_2.5-5kV-Shielded" H 4350 8950 50  0001 C CNN
 F 3 "https://www.xppower.com/Portals/0/pdfs/SF_Q_Series.pdf" H 4350 8950 50  0001 C CNN
 	1    4950 8750
@@
 F 0 "U6" H 2550 7517 50  0000 C CNN
 F 1 "EMCO-Q10-5" H 2550 7426 50  0000 C CNN
-F 2 "PPTBoard:EMCO_Q_2.5-5kV" H 1950 7250 50  0001 C CNN
+F 2 "PPTBoard:EMCO_Q_2.5-5kV-Shielded" H 1950 7250 50  0001 C CNN
 F 3 "https://www.xppower.com/Portals/0/pdfs/SF_Q_Series.pdf" H 1950 7250 50  0001 C CNN
 	1    2550 7050
@@
 Text GLabel 9850 8500 0    50   Input ~ 0
 U5_CS
-Text GLabel 7050 3650 0    50   Input ~ 0
+Text GLabel 8800 3850 2    50   Input ~ 0
 U5_CS
-Text GLabel 7050 3150 0    50   Input ~ 0
+Text GLabel 7050 3250 0    50   Input ~ 0
 U12_FAULT
 Text GLabel 7150 4850 0    50   Input ~ 0
 U14_EN
-Text GLabel 7050 3250 0    50   Input ~ 0
+Text GLabel 7050 3150 0    50   Input ~ 0
 U12_EN
 Text GLabel 7150 4950 0    50   Input ~ 0
@@
 Text GLabel 8550 1900 0    50   Input ~ 0
 U16_CS
-Text GLabel 7150 5350 0    50   Input ~ 0
+Text GLabel 7150 5250 0    50   Input ~ 0
 U16_CS
 Wire Wire Line
@@
 Text GLabel 1300 3350 0    50   Input ~ 0
 U8_ALERT
-Text GLabel 7050 2950 0    50   Input ~ 0
+Text GLabel 7050 4350 0    50   Input ~ 0
 U9_ALERT
 Text GLabel 2500 6200 1    50   Input ~ 0
@@
 Wire Wire Line
 	2500 6400 3050 6400
-Text GLabel 8800 3950 2    50   Input ~ 0
+Text GLabel 7050 3450 0    50   Input ~ 0
 SCLK
 Text GLabel 8550 1800 0    50   Input ~ 0
@@
 F 0 "U15" H 13750 5617 50  0000 C CNN
 F 1 "EMCO-Q50-5" H 13750 5526 50  0000 C CNN
-F 2 "PPTBoard:EMCO_Q_2.5-5kV" H 13150 5350 50  0001 C CNN
+F 2 "PPTBoard:EMCO_Q_2.5-5kV-Shielded" H 13150 5350 50  0001 C CNN
 F 3 "https://www.xppower.com/Portals/0/pdfs/SF_Q_Series.pdf" H 13150 5350 50  0001 C CNN
 	1    13750 5150
@@
 $EndComp
 Text GLabel 12200 8050 1    50   Input ~ 0
-U4_EN
-Text GLabel 7050 3450 0    50   Input ~ 0
 U4_EN
 Text GLabel 8800 4050 2    50   Input ~ 0
@@
 Wire Wire Line
 	1800 2300 1800 2400
-Text GLabel 7050 3950 0    50   Input ~ 0
+Text GLabel 7150 5050 0    50   Input ~ 0
 SCL2
 Text GLabel 10950 5350 0    50   Input ~ 0
@@
 Wire Wire Line
 	7300 4050 7050 4050
-Text GLabel 7050 4050 0    50   Input ~ 0
+Text GLabel 7150 5150 0    50   Input ~ 0
 SDA2
 Text GLabel 6200 5950 2    50   Input ~ 0
@@
 Text GLabel 7050 3050 0    50   Input ~ 0
 U10_ALERT
-Text GLabel 7150 5150 0    50   Input ~ 0
-SDA1
 $Comp
 L Device:R RSCL1
@@
 Wire Wire Line
 	7300 4950 7150 4950
-Text GLabel 7150 5050 0    50   Input ~ 0
-SCL1
 Wire Wire Line
 	7150 5050 7300 5050
@@
 Text GLabel 2900 1600 0    50   Input ~ 0
 VCC
-Text Label 1700 4850 0    50   ~ 0
-Thruster_Control
-Wire Wire Line
-	7050 2950 7300 2950
 Wire Wire Line
 	7150 4850 7300 4850
@@
 Text GLabel 14000 8200 1    50   Input ~ 0
 U3_EN
-Text GLabel 7050 3350 0    50   Input ~ 0
+Text GLabel 7000 2950 0    50   Input ~ 0
 U3_EN
-Wire Wire Line
-	7300 3350 7050 3350
 Wire Wire Line
 	7050 4250 7300 4250
@@
 Wire Wire Line
 	13350 3750 13400 3750
-Text GLabel 7150 5250 0    50   Input ~ 0
+Text GLabel 7150 5350 0    50   Input ~ 0
 THRUST_CONTROL
 Wire Wire Line
 	7150 5250 7300 5250
-Text GLabel 8800 3850 2    50   Input ~ 0
-U5_DIN
-Wire Wire Line
-	8800 3850 8700 3850
 Wire Notes Line
 	13800 7900 14150 7900
@@
 Wire Wire Line
 	5700 1600 5850 1600
+Text Label 1700 4850 0    50   ~ 0
+Thrust_Connector
+Wire Wire Line
+	7050 4350 7300 4350
+Wire Wire Line
+	7000 2950 7300 2950
+Wire Wire Line
+	7300 3350 7050 3350
+Wire Wire Line
+	8800 3850 8700 3850
+Text GLabel 7050 3350 0    50   Input ~ 0
+U5_DIN
+Text GLabel 8800 3950 2    50   Input ~ 0
+U4_EN
+Text GLabel 7050 3950 0    50   Input ~ 0
+SCL1
+Text GLabel 7050 4050 0    50   Input ~ 0
+SDA1
+Text GLabel 13750 5650 3    50   Input ~ 0
+GND
+Wire Wire Line
+	13750 5650 13750 5550
+Text GLabel 4950 9400 3    50   Input ~ 0
+GND
+Wire Wire Line
+	4950 9400 4950 9150
+Wire Wire Line
+	2550 7450 2550 7550
+Text GLabel 2550 7550 3    50   Input ~ 0
+GND
 $EndSCHEMATC
